File: board/bigtime.kicad_pcb (KiCad board)
At the start: 2 copper layers, 90 x 142 mm, 124 parts, among them IC1 NPIC6C596A, IC2 TPS62152, IC3 25AA02E48, IC4 STM32F407VET6, IC5 KSZ8081RNx, IC6 MAX5969x, IC7 MAX17503, IC8 LDL212DR, J1 RJHSE-538B, J2 MICROUSB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

Commit message: Removed MAC from silk
Other:
- board text removed: "MAC:"
Changed lines of the file:
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@@
     (area 124.744999 15.8125 215.4275 161.1725)
     (thickness 1.6)
-    (drawings 50)
+    (drawings 49)
     (tracks 1617)
     (zones 0)
@@
   )
   (gr_line (start 153.5 157) (end 153.5 157) (layer F.SilkS) (width 0.2))
-  (gr_text MAC: (at 138.5 151.5) (layer F.SilkS)
-    (effects (font (size 2 2) (thickness 0.3)))
-  )
   (gr_text r1 (at 138 156) (layer F.SilkS)
     (effects (font (size 2 2) (thickness 0.3)))
@@
       )
     )
-  )
-  (zone (net 0) (net_name "") (layer F.SilkS) (hatch full 0.508)
-    (connect_pads (clearance 0.508))
-    (min_thickness 0.254)
-    (fill yes (arc_segments 16) (thermal_gap 0.508) (thermal_bridge_width 0.508))
-    (polygon
-      (pts
-        (xy 142.5 149) (xy 142.5 153.5) (xy 152 153.5) (xy 152 149)
-      )
-    )
-  )
-  (zone (net 0) (net_name "") (layer F.SilkS) (hatch full 0.508)
-    (connect_pads (clearance 0.508))
-    (min_thickness 0.254)
-    (fill yes (arc_segments 16) (thermal_gap 0.508) (thermal_bridge_width 0.508))
-    (polygon
-      (pts
-        (xy 153 149) (xy 153 153.5) (xy 162.5 153.5) (xy 162.5 149)
-      )
-    )
-  )
-  (zone (net 0) (net_name "") (layer F.SilkS) (hatch full 0.508)
-    (connect_pads (clearance 0.508))
-    (min_thickness 0.254)
-    (fill yes (arc_segments 16) (thermal_gap 0.508) (thermal_bridge_width 0.508))
-    (polygon
-      (pts
-        (xy 163.5 149) (xy 163.5 153.5) (xy 173 153.5) (xy 173 149)
-      )
-    )
-  )
-  (zone (net 0) (net_name "") (layer F.SilkS) (hatch full 0.508)
-    (connect_pads (clearance 0.508))
-    (min_thickness 0.254)
-    (fill yes (arc_segments 16) (thermal_gap 0.508) (thermal_bridge_width 0.508))
-    (polygon
-      (pts
-        (xy 174 149) (xy 174 153.5) (xy 183.5 153.5) (xy 183.5 149)
-      )
-    )
-  )
-  (zone (net 0) (net_name "") (layer F.SilkS) (hatch full 0.508)
-    (connect_pads (clearance 0.508))
-    (min_thickness 0.254)
-    (fill yes (arc_segments 16) (thermal_gap 0.508) (thermal_bridge_width 0.508))
-    (polygon
-      (pts
-        (xy 184.5 149) (xy 184.5 153.5) (xy 194 153.5) (xy 194 149)
-      )
-    )
-  )
-  (zone (net 0) (net_name "") (layer F.SilkS) (hatch full 0.508)
-    (connect_pads (clearance 0.508))
-    (min_thickness 0.254)
-    (fill yes (arc_segments 16) (thermal_gap 0.508) (thermal_bridge_width 0.508))
-    (polygon
-      (pts
-        (xy 195 149) (xy 195 153.5) (xy 204.5 153.5) (xy 204.5 149)
-      )
-    )
