File: board/bigtime.sch (KiCad schematic (older format))
At the start: 61 parts, among them IC1 NPIC6C596A, IC2 TPS62152, IC3 25AA02E48, IC4 STM32F407VET6, IC8 LDL212DR, J2 MICROUSB, P1 CONN_IN, P2 CONN_OUT, P3 +12V, P4 SWD_TC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

Commit message: Final finishing touches and gerbers
Parts:
- removed P3: +12V, Connect:BARREL_JACK, symbol CONN_01X02
- added P3: +12V, Connect:BARREL_JACK, symbol CONN_01X03
- added TP6: GND, agg:SIL-254P-01, symbol TEST
- added X5: PART, Symbols:Polarity_Center_Positive_6mm_SilkScreen, symbol PART
- U1: value SA40-19 -> SA40-19SURKWA; Farnell (none) -> 2080056
Connections:
- net +12V: now also P3.1 (P1)
- net GND: now also P3.2 (P2), P3.3 (P3), TP6.1
Changed lines of the file:
@@
 P 10450 4500
 F 0 "U1" H 10350 5100 60  0000 L CNN
-F 1 "SA40-19" H 10200 3900 60  0000 L CNN
+F 1 "SA40-19SURKWA" H 10200 3900 60  0000 L CNN
 F 2 "footprints:SA40-18" H 2700 -650 60  0001 C CNN
-F 3 "" H 2700 -650 60  0001 C CNN
+F 3 "http://www.farnell.com/datasheets/2046843.pdf" H 2700 -650 60  0001 C CNN
+F 4 "2080056" H 10450 4500 60  0001 C CNN "Farnell"
 	1    10450 4500
 	1    0    0    -1
@@
 $EndSheet
 $Comp
-L CONN_01X02 P3
-U 1 1 58BC54A8
-P 7900 3000
-F 0 "P3" H 7819 2725 50  0000 C CNN
-F 1 "+12V" H 7819 2816 50  0000 C CNN
-F 2 "Connect:BARREL_JACK" H 7900 3000 50  0001 C CNN
-F 3 "" H 7900 3000 50  0000 C CNN
-	1    7900 3000
-	-1   0    0    1
-$EndComp
-$Comp
 L GND #PWR016
 U 1 1 58BC5CDB
-P 8100 3050
-F 0 "#PWR016" H 8100 2800 50  0001 C CNN
-F 1 "GND" V 8050 2850 50  0000 C CNN
-F 2 "" H 8100 3050 50  0000 C CNN
-F 3 "" H 8100 3050 50  0000 C CNN
-	1    8100 3050
+P 7550 2750
+F 0 "#PWR016" H 7550 2500 50  0001 C CNN
+F 1 "GND" V 7500 2550 50  0000 C CNN
+F 2 "" H 7550 2750 50  0000 C CNN
+F 3 "" H 7550 2750 50  0000 C CNN
+	1    7550 2750
 	0    -1   -1   0
 $EndComp
@@
 L +12V #PWR017
 U 1 1 58BC5F20
-P 8100 2950
-F 0 "#PWR017" H 8100 2800 50  0001 C CNN
-F 1 "+12V" V 8050 3150 50  0000 C CNN
-F 2 "" H 8100 2950 50  0000 C CNN
-F 3 "" H 8100 2950 50  0000 C CNN
-	1    8100 2950
+P 7400 2950
+F 0 "#PWR017" H 7400 2800 50  0001 C CNN
+F 1 "+12V" V 7350 3150 50  0000 C CNN
+F 2 "" H 7400 2950 50  0000 C CNN
+F 3 "" H 7400 2950 50  0000 C CNN
+	1    7400 2950
 	0    1    1    0
 $EndComp
@@
 $Comp
 L PWR_FLAG #FLG041
-U 0 1 58E0C1AE
+U 1 1 58E0C1AE
 P 10700 900
 F 0 "#FLG041" H 10700 975 50  0001 C CNN
@@
 F 2 "" H 10700 900 50  0001 C CNN
 F 3 "" H 10700 900 50  0001 C CNN
-	0    10700 900
+	1    10700 900
 	1    0    0    -1
 $EndComp
@@
 	10700 900  10700 1000
 Connection ~ 10700 1000
+$Comp
+L PART X5
+U 1 1 58E0EC81
+P 550 6900
+F 0 "X5" H 1078 6996 50  0000 L CNN
+F 1 "PART" H 1078 6905 50  0000 L CNN
+F 2 "Symbols:Polarity_Center_Positive_6mm_SilkScreen" H 550 6900 50  0001 C CNN
+F 3 "" H 550 6900 50  0001 C CNN
+	1    550  6900
+	1    0    0    -1
+$EndComp
+$Comp
+L CONN_01X03 P3
+U 1 1 58E160A2
+P 7050 2850
+F 0 "P3" H 6969 2525 50  0000 C CNN
+F 1 "+12V" H 6969 2616 50  0000 C CNN
+F 2 "Connect:BARREL_JACK" H 7050 2850 50  0001 C CNN
+F 3 "" H 7050 2850 50  0001 C CNN
+	1    7050 2850
+	-1   0    0    1
+$EndComp
+Wire Wire Line
+	7250 2750 7550 2750
+Wire Wire Line
+	7250 2950 7400 2950
+Wire Wire Line
+	7250 2850 7300 2850
+Wire Wire Line
+	7300 2850 7300 2750
+Connection ~ 7300 2750
+$Comp
+L TEST TP6
+U 1 1 58E2E95F
+P 7450 2650
+F 0 "TP6" H 7528 2790 50  0000 L CNN
+F 1 "GND" H 7528 2699 50  0000 L CNN
+F 2 "agg:SIL-254P-01" H 7450 2650 50  0001 C CNN
+F 3 "" H 7450 2650 50  0001 C CNN
+	1    7450 2650
+	1    0    0    -1
+$EndComp
+Wire Wire Line
+	7450 2650 7450 2750
+Connection ~ 7450 2750
 $EndSCHEMATC

Commit message: Order codes for capacitor shrapnel
Parts:
- C1, C10, C11, C12, C13, C14, C17, C18, C46, C5, C7, C9: Farnell (none) -> 2522597
- C15, C16: Farnell (none) -> 1735526
- C19, C20: Farnell (none) -> 2496912
- C21, C8: Farnell (none) -> 2611924
- C22, C6: Farnell (none) -> 1828801
- C44, C45: Farnell (none) -> 2496887
Changed lines of the file:
@@
 F 2 "agg:0603" H 2388 -100 50  0001 C CNN
 F 3 "" H 2350 50  50  0000 C CNN
+F 4 "2522597" H 6850 5250 60  0001 C CNN "Farnell"
 	1    6850 5250
 	-1   0    0    1
@@
 F 2 "agg:0603" H -162 300 50  0001 C CNN
 F 3 "" H -200 450 50  0001 C CNN
+F 4 "1828801" H 6800 4200 60  0001 C CNN "Farnell"
 	1    6800 4200
 	-1   0    0    1
@@
 F 2 "agg:0603" H 888 -200 50  0001 C CNN
 F 3 "" H 850 -50 50  0001 C CNN
+F 4 "2611924" H 8400 4150 60  0001 C CNN "Farnell"
 	1    8400 4150
 	1    0    0    -1
@@
 F 2 "agg:0603" H 1438 750 50  0001 C CNN
 F 3 "" H 1400 900 50  0000 C CNN
+F 4 "2522597" H 1400 900 60  0001 C CNN "Farnell"
 	1    1400 900
 	1    0    0    -1
@@
 F 2 "agg:0603" H 1788 750 50  0001 C CNN
 F 3 "" H 1750 900 50  0000 C CNN
+F 4 "1828801" H 1750 900 60  0001 C CNN "Farnell"
 	1    1750 900
 	1    0    0    -1
@@
 F 2 "agg:0603" H 2488 750 50  0001 C CNN
 F 3 "" H 2450 900 50  0000 C CNN
+F 4 "2611924" H 2450 900 60  0001 C CNN "Farnell"
 	1    2450 900
 	1    0    0    -1
@@
 F 2 "agg:0603" H 2138 750 50  0001 C CNN
 F 3 "" H 2100 900 50  0000 C CNN
+F 4 "2522597" H 2100 900 60  0001 C CNN "Farnell"
 	1    2100 900
 	1    0    0    -1
@@
 F 2 "agg:0603" H 2838 750 50  0001 C CNN
 F 3 "" H 2800 900 50  0000 C CNN
+F 4 "2522597" H 2800 900 60  0001 C CNN "Farnell"
 	1    2800 900
 	1    0    0    -1
@@
 F 2 "agg:0603" H 3138 750 50  0001 C CNN
 F 3 "" H 3100 900 50  0000 C CNN
+F 4 "2522597" H 3100 900 60  0001 C CNN "Farnell"
 	1    3100 900
 	1    0    0    -1
@@
 F 2 "agg:0603" H 3438 750 50  0001 C CNN
 F 3 "" H 3400 900 50  0000 C CNN
+F 4 "2522597" H 3400 900 60  0001 C CNN "Farnell"
 	1    3400 900
 	1    0    0    -1
@@
 F 2 "agg:0603" H 3738 750 50  0001 C CNN
 F 3 "" H 3700 900 50  0000 C CNN
+F 4 "2522597" H 3700 900 60  0001 C CNN "Farnell"
 	1    3700 900
 	1    0    0    -1
@@
 F 2 "agg:0603" H 4038 750 50  0001 C CNN
 F 3 "" H 4000 900 50  0000 C CNN
+F 4 "2522597" H 4000 900 60  0001 C CNN "Farnell"
 	1    4000 900
 	1    0    0    -1
@@
 F 2 "agg:0603" H 4338 750 50  0001 C CNN
 F 3 "" H 4300 900 50  0000 C CNN
+F 4 "2522597" H 4300 900 60  0001 C CNN "Farnell"
 	1    4300 900
 	1    0    0    -1
@@
 F 2 "agg:0603" H 1788 2800 50  0001 C CNN
 F 3 "" H 1750 2950 50  0000 C CNN
+F 4 "1735526" H 1750 2950 60  0001 C CNN "Farnell"
 	1    1750 2950
 	1    0    0    -1
@@
 F 2 "agg:0603" H 2038 2800 50  0001 C CNN
 F 3 "" H 2000 2950 50  0000 C CNN
+F 4 "1735526" H 2000 2950 60  0001 C CNN "Farnell"
 	1    2000 2950
 	1    0    0    -1
@@
 F 2 "agg:0603" H 838 3550 50  0001 C CNN
 F 3 "" H 800 3700 50  0000 C CNN
+F 4 "2522597" H 800 3700 60  0001 C CNN "Farnell"
 	1    800  3700
 	1    0    0    -1
@@
 F 2 "agg:0603" H 1538 3950 50  0001 C CNN
 F 3 "" H 1500 4100 50  0000 C CNN
+F 4 "2496912" H 1500 4100 60  0001 C CNN "Farnell"
 	1    1500 4100
 	1    0    0    -1
@@
 F 2 "agg:0603" H 1788 3950 50  0001 C CNN
 F 3 "" H 1750 4100 50  0000 C CNN
+F 4 "2496912" H 1750 4100 60  0001 C CNN "Farnell"
 	1    1750 4100
 	1    0    0    -1
@@
 F 2 "agg:0603" H 5088 3800 50  0001 C CNN
 F 3 "" H 5050 3950 50  0000 C CNN
+F 4 "2522597" H 5050 3950 60  0001 C CNN "Farnell"
 	1    5050 3950
 	1    0    0    -1
@@
 F 2 "agg:0603" H 4138 3200 50  0001 C CNN
 F 3 "" H 4100 3350 50  0001 C CNN
+F 4 "2496887" H 4100 3350 60  0001 C CNN "Farnell"
 	1    4100 3350
 	1    0    0    -1
@@
 F 2 "agg:0603" H 4388 3200 50  0001 C CNN
 F 3 "" H 4350 3350 50  0001 C CNN
+F 4 "2496887" H 4350 3350 60  0001 C CNN "Farnell"
 	1    4350 3350
 	1    0    0    -1
@@
 F 2 "agg:0603" H 8138 1000 50  0001 C CNN
 F 3 "" H 8100 1150 50  0001 C CNN
+F 4 "2522597" H 8100 1150 60  0001 C CNN "Farnell"
 	1    8100 1150
 	1    0    0    -1

Commit message: specced remaining parts
Parts:
- R29: Farnell (none) -> 9238603
- R30, R31: Farnell (none) -> 9238301
- TP6: symbol TEST -> TEST-RESCUE-bigtime
Changed lines of the file:
@@
 F 2 "agg:0603" V 6630 1150 50  0001 C CNN
 F 3 "" H 6700 1150 50  0001 C CNN
+F 4 "9238603" H 6700 1150 60  0001 C CNN "Farnell"
 	1    6700 1150
 	0    1    1    0
@@
 F 2 "agg:0603" H 2450 7250 50  0001 C CNN
 F 3 "" H 2450 7250 50  0000 C CNN
+F 4 "9238301" H 2450 7250 60  0001 C CNN "Farnell"
 	1    2450 7250
 	0    -1   -1   0
@@
 F 2 "agg:0603" H 2450 7150 50  0001 C CNN
 F 3 "" H 2450 7150 50  0000 C CNN
+F 4 "9238301" H 2450 7150 60  0001 C CNN "Farnell"
 	1    2450 7150
 	0    -1   -1   0
@@
 Connection ~ 7300 2750
 $Comp
-L TEST TP6
+L TEST-RESCUE-bigtime TP6
 U 1 1 58E2E95F
 P 7450 2650
